Commit message: Updating skratch_desription with new kelo stl

File: skratch_description/robots/skratch_config.urdf.xacro (robot description, xacro)
@@ -17,5 +17,5 @@
     <xacro:skratch_top_base name="skratch_left_top_base"/>
     <joint name="base_joint" type="fixed">
-        <origin xyz="0.0 0.0 0.02" rpy="0.0 0.0 0.0"/>
+        <origin xyz="0.0 0.0 0.025" rpy="0.0 0.0 0.0"/>
         <parent link="base_link"/>
         <child link="skratch_left_top_base"/>
@@ -23,5 +23,5 @@
     <xacro:skratch_top_base name="skratch_right_top_base"/>
     <joint name="right_top_base_joint" type="fixed">
-        <origin xyz="0.0 0.0 0.02" rpy="0.0 0.0 3.14"/>
+        <origin xyz="0.0 0.0 0.025" rpy="0.0 0.0 3.14"/>
         <parent link="base_link"/>
         <child link="skratch_right_top_base"/>
@@ -29,5 +29,5 @@
     <xacro:skratch_bottom_base name="skratch_left_bottom_base"/>
     <joint name="left_bottom_base_joint" type="fixed">
-        <origin xyz="0.0 -0.099 -0.138" rpy="3.14 0.0 0.0"/>
+        <origin xyz="0.0 -0.099 -0.148" rpy="3.14 0.0 0.0"/>
         <parent link="skratch_left_top_base"/>
         <child link="skratch_left_bottom_base"/>
@@ -35,5 +35,5 @@
     <xacro:skratch_bottom_base name="skratch_right_bottom_base"/>
     <joint name="right_bottom_base_joint" type="fixed">
-        <origin xyz="0.0 -0.099 -0.138" rpy="3.14 0.0 0.0"/>
+        <origin xyz="0.0 -0.099 -0.148" rpy="3.14 0.0 0.0"/>
         <parent link="skratch_right_top_base"/>
         <child link="skratch_right_bottom_base"/>
@@ -53,14 +53,14 @@
     <!-- Build wheels using kelo drive -->
     <xacro:kelo_drive name="wheel0" parent="skratch_right_wheel_support" movable_joints="$(arg movable_joints)">
-        <origin xyz="0.202 0.0 -0.09" rpy="0.0 0.0 0.0"/>
+        <origin xyz="0.178 0.0 -0.125" rpy="0.0 0.0 0.0"/>
     </xacro:kelo_drive>
     <xacro:kelo_drive name="wheel3" parent="skratch_left_wheel_support" movable_joints="$(arg movable_joints)">
-        <origin xyz="0.202 0.0 -0.09" rpy="0.0 0.0 0.0"/>
+        <origin xyz="0.178 0.0 -0.125" rpy="0.0 0.0 0.0"/>
     </xacro:kelo_drive>
     <xacro:kelo_drive name="wheel1" parent="skratch_right_wheel_support" movable_joints="$(arg movable_joints)">
-        <origin xyz="-0.202 0.0 -0.09" rpy="0.0 0.0 0.0"/>
+        <origin xyz="-0.178 0.0 -0.125" rpy="0.0 0.0 0.0"/>
     </xacro:kelo_drive>
     <xacro:kelo_drive name="wheel2" parent="skratch_left_wheel_support" movable_joints="$(arg movable_joints)">
-        <origin xyz="-0.202 0.0 -0.09" rpy="0.0 0.0 0.0"/>
+        <origin xyz="-0.178 0.0 -0.125" rpy="0.0 0.0 0.0"/>
     </xacro:kelo_drive>
     <!-- Build Front Lidar -->
@@ -70,9 +70,9 @@
             ros_topic="/front_scan"
             update_rate="10"
-            min_angle="-1.57"
-            max_angle="1.57" />
+            min_angle="0.0"
+            max_angle="-3.83" />
         <joint name="front_lidar_joint" type="fixed">
-            <origin xyz="0.320 -0.21 -0.165" rpy="0.0 0.0 0.81"/>
-            <parent link="skratch_left_top_base"/>
+            <origin xyz="0.320 -0.21 -0.160" rpy="0.0 0.0 0.81"/>
+            <parent link="skratch_right_top_base"/>
             <child link="front_lidar_link"/>
         </joint>
@@ -84,9 +84,9 @@
             ros_topic="/rear_scan"
             update_rate="10"
-            min_angle="-1.57"
-            max_angle="1.57" />
+            min_angle="0.0"
+            max_angle="-3.83" />
         <joint name="rear_lidar_joint" type="fixed">
-            <origin xyz="0.320 -0.205 -0.165" rpy="0.0 0.0 0.81"/>
-            <parent link="skratch_right_top_base"/>
+            <origin xyz="0.320 -0.205 -0.160" rpy="0.0 0.0 0.81"/>
+            <parent link="skratch_left_top_base"/>
             <child link="rear_lidar_link"/>
         </joint>

File: skratch_description/urdf/base_macros/kelo_drive.urdf.xacro (robot description, xacro)
@@ -3,29 +3,5 @@
 Copyright (c) 2021
 KELO Robotics GmbH
-Author:
-Sushant Chavan
-This software is published under a dual-license: GNU Lesser General Public
-License LGPL 2.1 and BSD license. The dual-license implies that users of this
-code may choose which terms they prefer.
-Redistribution and use in source and binary forms, with or without
-modification, are permitted provided that the following conditions are met:
-* Redistributions of source code must retain the above copyright
-notice, this list of conditions and the following disclaimer.
-* Redistributions in binary form must reproduce the above copyright
-notice, this list of conditions and the following disclaimer in the
-documentation and/or other materials provided with the distribution.
-* Neither the name of Locomotec nor the names of its
-contributors may be used to endorse or promote products derived from
-this software without specific prior written permission.
-This program is free software: you can redistribute it and/or modify
-it under the terms of the GNU Lesser General Public License LGPL as
-published by the Free Software Foundation, either version 2.1 of the
-License, or (at your option) any later version or the BSD license.
-This program is distributed in the hope that it will be useful,
-but WITHOUT ANY WARRANTY; without even the implied warranty of
-MERCHANTABILITY or FITNESS FOR A PARTICULAR PURPOSE. See the
-GNU Lesser General Public License LGPL and the BSD license for more details.
-You should have received a copy of the GNU Lesser General Public
-License LGPL and BSD license along with this program.
+Using kelo drive wheels with some modifications to suit skratch bot
 -->
 <robot xmlns:xacro="http://www.ros.org/wiki/xacro">
@@ -62,7 +38,7 @@
         <link name="${name}_pivot_link">
             <visual>
-                <origin xyz="0 0 0" rpy="0 0 0"/>
+                <origin xyz="-0.02 0.0 0.095" rpy="0 0 1.57"/>
                 <geometry>
-                    <mesh filename="file://$(find skratch_description)/meshes/kelo_drive/kelo_drive_base.dae" scale="1 1 1"/>
+                    <mesh filename="file://$(find skratch_description)/meshes/kelo_drive/kelo_drive_base_new.stl" scale="0.001 0.001 0.001"/>
                 </geometry>
             </visual>
