Commit message: [URDF]New base comibined stl

File: skratch_description/base/skratch_wheel_support.xacro (robot description, xacro)
@@ -9,5 +9,5 @@
             </inertial>
             <visual>
-                <origin xyz="0.0 0.0 0.0" rpy="0.0 0.0 0.0" />
+                <origin xyz="0.0 0.0 0.0" rpy="3.14 0.0 0.0" />
                 <geometry>
                     <mesh filename="file://$(find skratch_description)/meshes/base/skratch_wheel_support.stl" scale="0.001 0.001 0.001"/>
@@ -18,5 +18,5 @@
             </visual>
             <collision>
-                <origin xyz="0.0 0.0 0.0" rpy="0.0 0.0 0.0" />
+                <origin xyz="0.0 0.0 0.0" rpy="3.14 0.0 0.0" />
                 <geometry>
                     <mesh filename="file://$(find skratch_description)/meshes/base/skratch_wheel_support.stl" scale="0.001 0.001 0.001"/>

File: skratch_description/robots/skratch_config.urdf.xacro (robot description, xacro)
@@ -7,63 +7,31 @@
     <!-- Include base plate -->
     <xacro:include filename="$(find skratch_description)/base/skratch_base_plate.xacro" />
-    <xacro:include filename="$(find skratch_description)/base/skratch_bottom_base.xacro" />
-    <xacro:include filename="$(find skratch_description)/base/skratch_top_base.xacro" />
-    <xacro:include filename="$(find skratch_description)/base/skratch_wheel_support.xacro" />
     <!--Include Lidar-->
     <xacro:include filename="$(find skratch_description)/lidar/lidar_with_plugin.xacro" />
+    <xacro:include filename="$(find skratch_description)/base/skratch_base.xacro" />
     <!-- Start building the robot -->
     <link name="base_link"/>
-    <!-- Build base plate and joints -->
-    <xacro:skratch_top_base name="skratch_left_top_base"/>
-    <joint name="base_joint" type="fixed">
+    <!-- Skratch complete base-->
+   <xacro:skratch_base name="skratch_base"/>
+    <joint name="skratch_base_joint" type="fixed">
         <origin xyz="0.0 0.0 0.025" rpy="0.0 0.0 0.0"/>
         <parent link="base_link"/>
-        <child link="skratch_left_top_base"/>
-    </joint>
-    <xacro:skratch_top_base name="skratch_right_top_base"/>
-    <joint name="right_top_base_joint" type="fixed">
-        <origin xyz="0.0 0.0 0.025" rpy="0.0 0.0 3.14"/>
-        <parent link="base_link"/>
-        <child link="skratch_right_top_base"/>
-    </joint>
-    <xacro:skratch_bottom_base name="skratch_left_bottom_base"/>
-    <joint name="left_bottom_base_joint" type="fixed">
-        <origin xyz="0.0 -0.099 -0.148" rpy="3.14 0.0 0.0"/>
-        <parent link="skratch_left_top_base"/>
-        <child link="skratch_left_bottom_base"/>
-    </joint>
-    <xacro:skratch_bottom_base name="skratch_right_bottom_base"/>
-    <joint name="right_bottom_base_joint" type="fixed">
-        <origin xyz="0.0 -0.099 -0.148" rpy="3.14 0.0 0.0"/>
-        <parent link="skratch_right_top_base"/>
-        <child link="skratch_right_bottom_base"/>
-    </joint>
-    <xacro:skratch_wheel_support name="skratch_left_wheel_support"/>
-    <joint name="left_wheel_support_joint" type="fixed">
-        <origin xyz="0.0 -0.118 0" rpy="0.0 0.0 0.0"/>
-        <parent link="base_link"/>
-        <child link="skratch_left_wheel_support"/>
-    </joint>
-    <xacro:skratch_wheel_support name="skratch_right_wheel_support"/>
-    <joint name="right_wheel_support_joint" type="fixed">
-        <origin xyz="0.0 0.118 0.0" rpy="0.0 0.0 0.0"/>
-        <parent link="base_link"/>
-        <child link="skratch_right_wheel_support"/>
+        <child link="skratch_base"/>
     </joint>
     <!-- Build wheels using kelo drive -->
-    <xacro:kelo_drive name="wheel0" parent="skratch_right_wheel_support" movable_joints="$(arg movable_joints)">
-        <origin xyz="0.178 0.0 -0.125" rpy="0.0 0.0 0.0"/>
+    <xacro:kelo_drive name="wheel0" parent="skratch_base" movable_joints="$(arg movable_joints)">
+        <origin xyz="0.180 0.118 0.0" rpy="0.0 0.0 3.14"/>
     </xacro:kelo_drive>
-    <xacro:kelo_drive name="wheel3" parent="skratch_left_wheel_support" movable_joints="$(arg movable_joints)">
-        <origin xyz="0.178 0.0 -0.125" rpy="0.0 0.0 0.0"/>
+    <xacro:kelo_drive name="wheel1" parent="skratch_base" movable_joints="$(arg movable_joints)">
+        <origin xyz="-0.180 0.118 0.0" rpy="0.0 0.0 0.0"/>
     </xacro:kelo_drive>
-    <xacro:kelo_drive name="wheel1" parent="skratch_right_wheel_support" movable_joints="$(arg movable_joints)">
-        <origin xyz="-0.178 0.0 -0.125" rpy="0.0 0.0 0.0"/>
+    <xacro:kelo_drive name="wheel3" parent="skratch_base" movable_joints="$(arg movable_joints)">
+        <origin xyz="0.180 -0.118 0.0" rpy="0.0 0.0 3.14"/>
     </xacro:kelo_drive>
-    <xacro:kelo_drive name="wheel2" parent="skratch_left_wheel_support" movable_joints="$(arg movable_joints)">
-        <origin xyz="-0.178 0.0 -0.125" rpy="0.0 0.0 0.0"/>
+    <xacro:kelo_drive name="wheel2" parent="skratch_base" movable_joints="$(arg movable_joints)">
+        <origin xyz="-0.180 -0.118 0.0" rpy="0.0 0.0 0.0"/>
     </xacro:kelo_drive>
     <!-- Build Front Lidar -->
-    <xacro:if value="$(arg use_sim)">
+    <!-- <xacro:if value="$(arg use_sim)">
         <xacro:lidar_with_plugin
             name="front_lidar"
@@ -73,11 +41,11 @@
             max_angle="-3.83" />
         <joint name="front_lidar_joint" type="fixed">
-            <origin xyz="0.320 -0.21 -0.160" rpy="0.0 0.0 0.81"/>
-            <parent link="skratch_right_top_base"/>
+            <origin xyz="0.320 -0.21 0.060" rpy="0.0 0.0 0.81"/>
+            <parent link="base_link"/>
             <child link="front_lidar_link"/>
         </joint>
-    </xacro:if>
+    </xacro:if> -->
     <!-- Build Rear Lidar -->
-    <xacro:if value="$(arg use_sim)">
+    <!-- <xacro:if value="$(arg use_sim)">
         <xacro:lidar_with_plugin
             name="rear_lidar"
@@ -87,20 +55,21 @@
             max_angle="-3.83" />
         <joint name="rear_lidar_joint" type="fixed">
-            <origin xyz="0.320 -0.205 -0.160" rpy="0.0 0.0 0.81"/>
-            <parent link="skratch_left_top_base"/>
+            <origin xyz="-0.320 0.22 0.060" rpy="0.0 0.0 0.81"/>
+            <parent link="base_link"/>
             <child link="rear_lidar_link"/>
         </joint>
-    </xacro:if>
-    <!-- Battery -->
-    <xacro:skratch_base_plate name="skratch_battery_base_plate"/>
-    <joint name="battery_base_plate_joint" type="fixed">
-        <origin xyz="-0.2115 0.005 0.023" rpy="0.0 0.0 3.1416"/>
-        <parent link="skratch_left_top_base"/>
-        <child link="skratch_battery_base_plate"/>
+    </xacro:if> -->
+    <!-- Arm plate -->
+    <xacro:skratch_base_plate name="skratch_arm_plate"/>
+    <joint name="skratch_arm_plate_joint" type="fixed">
+        <origin xyz="0.211 0.0 0.155" rpy="0.0 0.0 0.0"/>
+        <parent link="skratch_base"/>
+        <child link="skratch_arm_plate"/>
     </joint>
-    <link name="battery_link">
+    <!--Battery-->
+    <link name="battery_link_1">
         <visual>
             <geometry>
-                <box size="0.166 0.196 0.175"/>
+                <box size="0.166 0.166 0.175"/>
             </geometry>
             <material name="battery_color">
@@ -110,5 +79,5 @@
         <collision>
             <geometry>
-                <box size="0.166 0.196 0.175"/>
+                <box size="0.166 0.166 0.175"/>
             </geometry>
         </collision>
@@ -119,11 +88,40 @@
         </inertial>
     </link>
-    <gazebo reference="battery_link">
+    <gazebo reference="battery_link_1">
         <material>Gazebo/Black</material>
     </gazebo>
-    <joint name="battery_joint" type="fixed">
-        <origin xyz="0.0 0.0 0.0875" rpy="0.0 0.0 0.0"/>
-        <parent link="skratch_battery_base_plate"/>
-        <child link="battery_link"/>
+    <joint name="battery_joint_1" type="fixed">
+        <origin xyz="-0.200 -0.09 0.225" rpy="0.0 0.0 0.0"/>
+        <parent link="skratch_base"/>
+        <child link="battery_link_1"/>
+        <axis xyz="0.0 0.0 1.0"/>
+    </joint>
+    <link name="battery_link_2">
+        <visual>
+            <geometry>
+                <box size="0.166 0.166 0.175"/>
+            </geometry>
+            <material name="battery_color">
+                <color rgba="0.0 0.0 0.0 1.0"/>
+            </material>
+        </visual>
+        <collision>
+            <geometry>
+                <box size="0.166 0.166 0.175"/>
+            </geometry>
+        </collision>
+        <inertial>
+            <origin xyz="0 0 0" rpy="0 0 0"/>
+            <mass value="7.0"/>
+            <inertia ixx="0.403" ixy="0.0" ixz="0.0" iyy="0.345" iyz="0.0" izz="0.388"/>
+        </inertial>
+    </link>
+    <gazebo reference="battery_link_2">
+        <material>Gazebo/Black</material>
+    </gazebo>
+    <joint name="battery_joint_2" type="fixed">
+        <origin xyz="-0.200 0.095 0.225" rpy="0.0 0.0 0.0"/>
+        <parent link="skratch_base"/>
+        <child link="battery_link_2"/>
         <axis xyz="0.0 0.0 1.0"/>
     </joint>
