Commit message: Updating properly

File: skratch_description/base/skratch_base.xacro (robot description, xacro)
@@ -1,3 +1,10 @@
 <?xml version="1.0"?>
+<!--
+Copyright (c) 2025
+b-it-bots
+Hochschule Bonn-Rhein-Sieg
+Authors:
+Chaitanya Gumudala
+-->
 <robot name="skratch_base" xmlns:xacro="http://www.ros.org/wiki/xacro">
     <xacro:macro name="skratch_base" params="name">
@@ -5,5 +12,5 @@
             <inertial>
                 <mass value="2.0"/>
-                <origin xyz="0 0 0" rpy="0 0 0"/>
+                <origin xyz="0 0 -0.075" rpy="0 0 0"/>
                 <inertia ixx="0.03287973" iyy="0.06900190" izz="0.09325417" ixy="0.0" ixz="0.0" iyz="0.0"/>
             </inertial>
