Commit message: [skratch_description] Cleaning up

File: skratch_description/urdf/base_macros/kelo_drive_mid.urdf.xacro (robot description, xacro)
@@ -16,5 +16,4 @@
                 <parent link="${parent}"/>
                 <child link="${name}_pivot_link" />
-                <limit effort="2.0" velocity="1.0"/>
             </joint>
             <transmission name="${name}_pivot_transmission">
@@ -56,6 +55,4 @@
                 <inertia ixx="0.00302046423" ixy="0.00000851844" ixz="0.00001188180" iyy="0.00326495472" iyz="0.00001855408" izz="0.00386072964"/>
             </inertial>
-            <!--TODO: Set the correct inertia-->
-            <!-- <xacro:cuboid_inertia mass="10.0" length="0.233" breadth="0.233" height="0.233"/> -->
         </link>
         <!-- LEFT HUB WHEEL -->

File: skratch_description/urdf/base_macros/kelo_drive_wheel.urdf.xacro (robot description, xacro)
@@ -76,7 +76,4 @@
                 <inertia ixx="0.00101253363" ixy="0.00000000000" ixz="0.00000001020" iyy="0.00157998524" iyz="-0.00000055474" izz="0.00101282739"/>
             </inertial>
-            <!-- <xacro:cylinder_inertia mass="0.5" radius="0.0515" length="0.035" center_of_mass_roll="1.570796327"/> -->
-            <!--HACK: Use large cuboid inertias to fix the issue that the model breaks when JointVelocity controller is activated -->
-            <!-- <xacro:cuboid_inertia mass="10.0" length="0.233" breadth="0.233" height="0.233"/> -->
         </link>
     </xacro:macro>
