Commit message: [URDF] Updating urdf

File: skratch_description/gazebo/gazebo_skratch.xacro (robot description, xacro)
@@ -4,5 +4,5 @@
     <xacro:arg name="use_sim" default="true"/>
     <!-- Include desired kelo wheels -->
-    <xacro:include filename="$(find skratch_description)/urdf/base_macros/kelo_drive.urdf.xacro" />
+    <xacro:include filename="$(find skratch_description)/urdf/base_macros/kelo_drive_top.urdf.xacro" />
     <!--Include skratch base stl-->
      <xacro:include filename="$(find skratch_description)/base/skratch_base.xacro" />
@@ -16,21 +16,21 @@
    <xacro:skratch_base name="skratch_base"/>
     <joint name="skratch_base_joint" type="fixed">
-        <origin xyz="0.0 0.0 0.025" rpy="0.0 0.0 0.0"/>
+        <origin xyz="0.0 0.0 0" rpy="0.0 0.0 0.0"/>
         <parent link="base_link"/>
         <child link="skratch_base"/>
     </joint>
     <!-- Build wheels using kelo drive -->
-    <xacro:kelo_drive name="wheel0" parent="skratch_base" movable_joints="$(arg movable_joints)">
-        <origin xyz="0.180 0.118 0.0" rpy="0.0 0.0 3.14"/>
-    </xacro:kelo_drive>
-    <xacro:kelo_drive name="wheel1" parent="skratch_base" movable_joints="$(arg movable_joints)">
-        <origin xyz="-0.180 0.118 0.0" rpy="0.0 0.0 0.0"/>
-    </xacro:kelo_drive>
-    <xacro:kelo_drive name="wheel3" parent="skratch_base" movable_joints="$(arg movable_joints)">
-        <origin xyz="0.180 -0.118 0.0" rpy="0.0 0.0 3.14"/>
-    </xacro:kelo_drive>
-    <xacro:kelo_drive name="wheel2" parent="skratch_base" movable_joints="$(arg movable_joints)">
-        <origin xyz="-0.180 -0.118 0.0" rpy="0.0 0.0 0.0"/>
-    </xacro:kelo_drive>
+    <xacro:kelo_drive_top name="wheel0" parent="skratch_base" movable_joints="$(arg movable_joints)">
+        <origin xyz="0.190 0.118 0.0" rpy="0.0 0.0 0.0"/>
+    </xacro:kelo_drive_top>
+    <xacro:kelo_drive_top name="wheel1" parent="skratch_base" movable_joints="$(arg movable_joints)">
+        <origin xyz="-0.190 0.118 0.0" rpy="0.0 0.0 0.0"/>
+    </xacro:kelo_drive_top>
+    <xacro:kelo_drive_top name="wheel3" parent="skratch_base" movable_joints="$(arg movable_joints)">
+        <origin xyz="0.190 -0.118 0.0" rpy="0.0 0.0 0.0"/>
+    </xacro:kelo_drive_top>
+    <xacro:kelo_drive_top name="wheel2" parent="skratch_base" movable_joints="$(arg movable_joints)">
+        <origin xyz="-0.190 -0.118 0.0" rpy="0.0 0.0 0.0"/>
+    </xacro:kelo_drive_top>
     <!-- Build Front Lidar -->
     <!-- <xacro:if value="$(arg use_sim)">
@@ -62,12 +62,12 @@
     </xacro:if> -->
     <!-- Arm plate -->
-    <xacro:skratch_base_plate name="skratch_arm_plate"/>
+    <!-- <xacro:skratch_base_plate name="skratch_arm_plate"/>
     <joint name="skratch_arm_plate_joint" type="fixed">
         <origin xyz="0.211 0.0 0.155" rpy="0.0 0.0 0.0"/>
         <parent link="skratch_base"/>
         <child link="skratch_arm_plate"/>
-    </joint>
+    </joint> -->
     <!--Battery-->
-    <link name="battery_link_1">
+    <!-- <link name="battery_link_1">
         <visual>
             <geometry>
@@ -126,5 +126,5 @@
         <child link="battery_link_2"/>
         <axis xyz="0.0 0.0 1.0"/>
-    </joint>
+    </joint> -->
     <!-- Gazebo Plugins -->
     <xacro:if value="$(arg movable_joints)">

File: skratch_description/urdf/base_macros/kelo_drive_wheel.urdf.xacro (robot description, xacro)
@@ -62,16 +62,21 @@
                 <origin xyz="0 0 0" rpy="0 0 0"/>
                 <geometry>
-                    <mesh filename="file://$(find skratch_description)/meshes/kelo_drive/kelo_drive_wheel.dae" scale="1 1 1"/>
+                    <mesh filename="file://$(find skratch_description)/meshes/kelo_drive/kelo_drive_wheel.stl" scale="1 1 1"/>
                 </geometry>
             </visual>
             <collision>
-                <origin xyz="0 0 0" rpy="1.570796327 0 0"/>
+                <origin xyz="0 0 0" rpy="0 0 0"/>
                 <geometry>
-                    <cylinder radius="0.0515" length="0.035"/>
+                    <mesh filename="file://$(find skratch_description)/meshes/kelo_drive/kelo_drive_wheel.stl" scale="1 1 1"/>
                 </geometry>
             </collision>
+             <inertial>
+                <origin xyz="0 0 0" rpy="0 0 0"/>
+                <mass value="1.56317"/>
+                <inertia ixx="0.00101253363" ixy="0.00000000000" ixz="0.00000001020" iyy="0.00157998524" iyz="-0.00000055474" izz="0.00101282739"/>
+            </inertial>
             <!-- <xacro:cylinder_inertia mass="0.5" radius="0.0515" length="0.035" center_of_mass_roll="1.570796327"/> -->
             <!--HACK: Use large cuboid inertias to fix the issue that the model breaks when JointVelocity controller is activated -->
-            <xacro:cuboid_inertia mass="10.0" length="0.233" breadth="0.233" height="0.233"/>
+            <!-- <xacro:cuboid_inertia mass="10.0" length="0.233" breadth="0.233" height="0.233"/> -->
         </link>
     </xacro:macro>

Commit message: Update skratch configs

File: skratch_description/gazebo/gazebo_skratch.xacro (robot description, xacro)
@@ -2,5 +2,5 @@
 <robot xmlns:xacro="http://ros.org/wiki/xacro" name="skratch_platform_gazebo">
     <xacro:arg name="movable_joints" default="false" />
-    <xacro:arg name="use_sim" default="true"/>
+    <xacro:arg name="use_sim" default="false"/>
     <!-- Include desired kelo wheels -->
     <xacro:include filename="$(find skratch_description)/urdf/base_macros/kelo_drive_top.urdf.xacro" />
@@ -34,5 +34,5 @@
     </xacro:kelo_drive_top>
     <!-- Build Front Lidar -->
-    <!-- <xacro:if value="$(arg use_sim)">
+    <xacro:if value="$(arg use_sim)">
         <xacro:lidar_with_plugin
             name="front_lidar"
@@ -42,11 +42,11 @@
             max_angle="-3.83" />
         <joint name="front_lidar_joint" type="fixed">
-            <origin xyz="0.320 -0.21 0.060" rpy="0.0 0.0 0.81"/>
+            <origin xyz="0.320 -0.21 0.060" rpy=" 3.14 0.0 0.81"/>
             <parent link="base_link"/>
             <child link="front_lidar_link"/>
         </joint>
-    </xacro:if> -->
+    </xacro:if>
     <!-- Build Rear Lidar -->
-    <!-- <xacro:if value="$(arg use_sim)">
+    <xacro:if value="$(arg use_sim)">
         <xacro:lidar_with_plugin
             name="rear_lidar"
@@ -56,9 +56,9 @@
             max_angle="-3.83" />
         <joint name="rear_lidar_joint" type="fixed">
-            <origin xyz="-0.320 0.22 0.060" rpy="0.0 0.0 0.81"/>
+            <origin xyz="-0.320 0.22 0.060" rpy="3.14 0.0 0.81"/>
             <parent link="base_link"/>
             <child link="rear_lidar_link"/>
         </joint>
-    </xacro:if> -->
+    </xacro:if>
     <!-- Arm plate -->
     <!-- <xacro:skratch_base_plate name="skratch_arm_plate"/>

File: skratch_description/urdf/sensors/lidar_with_plugin.xacro (robot description, xacro)
@@ -5,5 +5,5 @@
     <link name="${name}_link">
       <inertial>
-        <origin xyz="0.0 0.0 0.027537" rpy="0.0 0.0 0.0" />
+        <origin xyz="0.0 0.0 0.027537" rpy="3.14 0.0 0.0" />
         <mass value="0.1" />
         <inertia ixx="0.00006111" iyy="0.00004167" izz="0.00006111" ixy="0.0" iyz="0.0" ixz="0.0" />
@@ -19,5 +19,5 @@
       </visual>
       <collision>
-        <origin xyz="0.0 0.0 0.6" rpy="0.0 3.14 0.0" />
+        <origin xyz="0.0 0.0 0.6" rpy="3.14 0.0 0.0" />
         <geometry>
           <mesh filename="file://$(find skratch_description)/meshes/lidar/lidar.stl" scale="0.001 0.001 0.001"/>
